File: untitled.kicad_sch (KiCad schematic)
At the start: 10 parts, among them J1 Conn_01x03_Pin

Commit message: fans
Other:
- note added: "TP7 to pull low if needed"
Changed lines of the file:
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@@
+		)
+	)
+	(text "TP7 to pull low if needed"
+		(exclude_from_sim no)
+		(at 327.152 263.652 0)
+		(effects
+			(font
+				(size 1.27 1.27)
+			)
 		)
 	)
