File: Carrier_Board.kicad_sch (KiCad schematic)
At the start: 0 parts

Commit message: changes to PSU
Parts:
- added FID1, FID2: Fiducial, symbol Mechanical:Fiducial
- added H1, H2, H3, H4: MountingHole_Pad, symbol Mechanical:MountingHole_Pad
Connections:
- new net GND: H1.1, H2.1, H3.1, H4.1
Other:
- added sheet Fan (Fan.kicad_sch)
- added sheet GPIO (GPIO.kicad_sch)
- added sheet Gagabit Eithernet (Gagabit_Eithernet.kicad_sch)
- added sheet HDMI (HDMI.kicad_sch)
- added sheet Latte_PandaMU (untitled.kicad_sch)
- added sheet PCIE x4 (PCIEx4.kicad_sch)
- added sheet PWR_supply (PWR_supply.kicad_sch)
- added sheet USB 2.0 & 3.0 (USB2&3.kicad_sch)
- added sheet m.2 M Key (m2_em.kicad_sch)

Commit message: fans
Other:
- sheet PWR_supply ports: added SLS_S3, ~{PWR_LED}/~{PSON}, ~{PWR_SW}, ~{RST_SW}; removed none
- moved on the sheet: FID1, FID2, H1, H2, H3, H4

Commit message: done with Fan
Other:
- sheet Fan ports: added FAN_1_PWM, FAN_1_TAC; removed none
Changed lines of the file:
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@@
+	(wire
+		(pts
+			(xy 185.42 250.19) (xy 212.09 250.19)
+		)
+		(stroke
+			(width 0)
+			(type default)
+		)
+	)
 	(wire
 		(pts
 			(xy 185.42 224.79) (xy 212.09 224.79)
+		)
+		(stroke
+			(width 0)
+			(type default)
+		)
+	)
+	(wire
+		(pts
+			(xy 185.42 245.11) (xy 212.09 245.11)
 		)
 		(stroke
@@
 		)
 		(pin "FAN_1_PWM" output
-			(at 121.285 146.685 180)
-			(effects
-				(font
-					(size 1.27 1.27)
-				)
-				(justify left)
+			(at 185.42 245.11 0)
+			(effects
+				(font
+					(size 1.27 1.27)
+				)
+				(justify right)
 			)
 		)
 		(pin "FAN_1_TAC" input
-			(at 121.285 149.225 180)
-			(effects
-				(font
-					(size 1.27 1.27)
-				)
-				(justify left)
+			(at 185.42 250.19 0)
+			(effects
+				(font
+					(size 1.27 1.27)
+				)
+				(justify right)
 			)
 		)
@@
 	)
 	(sheet
-		(at 491.49 245.11)
-		(size 39.37 31.75)
+		(at 212.09 242.57)
+		(size 27.94 11.43)
 		(exclude_from_sim no)
 		(in_bom yes)
@@
 		)
 		(property "Sheetname" "Fan"
-			(at 491.49 244.3984 0)
+			(at 212.09 241.8584 0)
 			(effects
 				(font
@@
 		)
 		(property "Sheetfile" "Fan.kicad_sch"
-			(at 491.49 277.4446 0)
+			(at 212.09 254.5846 0)
 			(effects
 				(font
@@
 			)
 		)
+		(pin "FAN_1_PWM" input
+			(at 212.09 245.11 180)
+			(effects
+				(font
+					(size 1.27 1.27)
+				)
+				(justify left)
+			)
+		)
+		(pin "FAN_1_TAC" output
+			(at 212.09 250.19 180)
+			(effects
+				(font
+					(size 1.27 1.27)
+				)
+				(justify left)
+			)
+		)
