File: Fan.kicad_sch (KiCad schematic)
At the start: 0 parts

Commit message: done with Fan
Parts:
- added C1: 100n, A_HDJ_Library:C_0402_1005Metric, symbol Device:C
- added D1: 1N5819, A_DFRobot:D_SOD-323, symbol Diode:1N5819WS
- added M1: Fan_4pin, A_HDJ_Library:JST_PH_B4B-PH-K_1x04_P2.00mm_Vertical, symbol Motor:Fan_4pin
- added R5: 20k, A_DFRobot:R_0402, symbol Device:R
- added R6: 100, A_DFRobot:R_0402, symbol Device:R
- added R8: 4.7k, A_DFRobot:R_0402, symbol Device:R
- added TP11, TP12: TestPoint, A_HDJ_Library:TestPoint_Pad_D1.5mm, symbol Connector:TestPoint
Connections:
- new net: M1.4 (PWM), R6.2
- new net: D1.2 (A), M1.3 (Tacho), R5.1, R8.2
- new net +5V_FAN: C1.1, D1.1 (K), M1.2 (+), R8.1
- new net FAN_1_PWM: R6.1, TP12.1
- new net FAN_1_TAC: R5.2, TP11.1
- new net GND: C1.2, M1.1 (-)
Other:
- note added: "LattePanda Mu has integrated pull-up resistors."
