File: PWR_supply.kicad_sch (KiCad schematic)
At the start: 12 parts, among them J17 Barrel_Jack_Switch_Pin3Ring, J18 USB_C_Receptacle_USB2.0_16P, U14 CH224K

Commit message: added more to PSU
Parts:
- added D15, D16, D17, D18, D19, D20: D_Schottky, Diode_SMD:D_SMA, symbol Device:D_Schottky
- added Q7: AON7262E, Package_DFN_QFN:DFN-8-1EP_3x3mm_P0.65mm_EP1.7x2.05mm, symbol AON7262E:AON7262E
- added TP10, TP3, TP4: TestPoint, symbol Connector:TestPoint
- renumbered R3 to R43
Connections:
- net +15V: now also D18.2 (A), D19.2 (A), D20.2 (A), TP3.1
- net GND: now also J17.2, J17.3
- net +12V: now reaches J17.1
- net +12V: now also D15.2 (A), D16.2 (A), D17.2 (A), TP4.1
- new net: D15.1 (K), D16.1 (K), D17.1 (K), D18.1 (K), D19.1 (K), D20.1 (K), TP10.1
Other:
- note added: "ESD5V0B03"
- note added: "R43 resistor can be changed if you want to request a different voltage(24k = 12V) CFG2 and 3 cant be connected in resistance config mode."
- note removed: "56k resistor can be changed if you want to request a different voltage(24k = 12V) CFG2 and 3 cant be connected in resistance config mode."
- moved on the sheet: J17

Commit message: more PSU
Parts:
- removed Q7: AON7262E, Package_DFN_QFN:DFN-8-1EP_3x3mm_P0.65mm_EP1.7x2.05mm, symbol AON7262E:AON7262E
- added C1, C3, C8, C9: .1u, symbol Device:C
- added C10, C11, C13, C14, C5, C6: 22u, symbol Device:C
- added C12: 47p, symbol Device:C
- added C2: 75p, symbol Device:C
- added C4, C7: 10u, symbol Device:C
- added L1: 10u, symbol Device:L
- added L2: 6.8u, symbol Device:L
- added R10, R7: 49.9, symbol Device:R
- added R11, R3, R5: 100k, symbol Device:R
- added R12: 22k, symbol Device:R
- added R4: 13.5k, symbol Device:R
- added R6: 100, symbol Device:R
- added U1, U2: TPS54302, Package_TO_SOT_SMD:SOT-23-6, symbol Regulator_Switching:TPS54302
Connections:
- net GND: now also C1.2, C10.2, C11.2, C13.2, C14.2, C4.2, C5.2, C6.2, C7.2, C8.2, R12.2, R4.2, R5.2, U1.1 (GND), U2.1 (GND)
- net at D15.1 (K), D16.1 (K), D17.1 (K)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: now also C1.1, C4.1, U1.3 (VIN)
- new net: C2.1, R3.1, R7.2
- new net: C2.2, R3.2, R4.1, U1.4 (FB)
- new net: C3.1, U1.6 (BOOT)
- new net: C3.2, L1.1, U1.2 (SW)
- new net: C10.1, C11.1, C13.1, L2.2, R10.1
- new net: C9.2, L2.1, U2.2 (SW)
- new net: C7.1, C8.1, U2.3 (VIN)
- new net: C12.1, R10.2, R11.1
- new net: C14.1, C5.1, C6.1, L1.2, R7.1
- new net: C12.2, R11.2, R12.1, U2.4 (FB)
- new net: C9.1, U2.6 (BOOT)
- new net EN: R5.1, R6.2, U1.5 (EN), U2.5 (EN)
Other:
- note added: "Using 3.3 =.596*(100k/R2 + 1), I get R2 = around 22k"
- note added: "Using 5=.596*(100k/R2 + 1), I get R2 = around 13.5k"
- moved on the sheet: D15, D16, D17, D18, D19, D20, J17, TP10, TP3, TP4

Commit message: fans
Parts:
- added C66, C69: 1uF/16V, A_HDJ_Library:C_0402_1005Metric, symbol Device:C
- added D21, D25: ESD5V0B03, A_HDJ_Library:D_0402_1005Metric, symbol Diode:ESD9B5.0ST5G
- added D22: LED_G, A_HDJ_Library:LED_0603_1608Metric, symbol Device:LED
- added D24: 3.3V, A_HDJ_Library:D_SOD-323, symbol Device:D_Schottky
- added JP1: Jumper_3_Bridged12, A_HDJ_Library:PinHeader_1x03_P2.54mm_Vertical, symbol Jumper:Jumper_3_Bridged12
- added Q8: 2N7002, A_HDJ_Library:SOT-23, symbol Transistor_FET:2N7002
- added R47: 1k, A_HDJ_Library:R_0402_1005Metric, symbol Device:R
- added R48, R55: 100R/1%, A_HDJ_Library:R_0402_1005Metric, symbol Device:R
- added R49: 10k, A_HDJ_Library:R_0402_1005Metric, symbol Device:R
- added R52, R53: 2.2k, A_HDJ_Library:R_0402_1005Metric, symbol Device:R
- added SW1, SW2: SW_Push, A_HDJ_Library:SW_Push_6x6x6, symbol Switch:SW_Push
- added TP13, TP5, TP6: TestPoint, A_HDJ_Library:TestPoint_Pad_D1.5mm, symbol Connector:TestPoint
- renumbered C4 to C64, C7 to C65, C1 to C67, C8 to C68, R6 to R46, R5 to R51
Connections:
- net GND: now also C66.2, C69.2, D21.1 (A1), D24.2 (A), D25.1 (A1), Q8.2 (S), R49.1, SW1.2, SW2.2
- net VDC: now reaches C64.1, C67.1, D15.1 (K), D16.1 (K), D17.1 (K), D18.1 (K), D19.1 (K), D20.1 (K), TP10.1, U1.3 (VIN)
- net VDC: now also C65.1, C68.1, U2.3 (VIN), R53.1
- net +3.3V: now reaches C10.1, C11.1, C13.1, L2.2, R10.1
- net +3.3V: now also TP6.1
- net +5V: now reaches C14.1, C5.1, C6.1, L1.2, R7.1
- net +5V: now also TP5.1
- net at R46.1: now also JP1.2 (C)
- net EN renamed PWR_EN
- new net: Q8.1 (G), R47.2, R49.2
- new net: D22.1 (K), Q8.3 (D)
- new net: D22.2 (A), R52.1
- new net +3V3: C66.1, C69.1, D21.2 (A2), D25.2 (A2), R48.1, R52.2, R55.1, SW1.1, SW2.1
- new net SLS_S3: JP1.3 (B)
- new net VPullup: D24.1 (K), R53.2, TP13.1
- new net ~{PWR_LED}/~{PSON}: JP1.1 (A), R47.1
- new net ~{PWR_SW}: R48.2
- new net ~{RST_SW}: R55.2
Other:
- note added: "12V input"
- note added: "15V input"
- note added: "LattePanda Mu has integrated pull-up resistors already"
- note added: "Pullup power for bios_sel"
- moved on the sheet: C10, C11, C12, C13, C14, C2, C3, C5, C6, C64, C65, C67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

Commit message: done with Fan
Connections:
- net +3V3: no longer C66.1, C69.1, D21.2 (A2), D25.2 (A2), R48.1, R55.1, SW1.1, SW2.1
- new net: C66.1, D21.2 (A2), R48.1, SW1.1
- new net: C69.1, D25.2 (A2), R55.1, SW2.1
Changed lines of the file:
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@@
 	(text "LattePanda Mu has integrated pull-up resistors already"
 		(exclude_from_sim no)
-		(at 320.04 322.58 0)
+		(at 273.812 327.152 0)
 		(effects
 			(font
@@
 	(wire
 		(pts
-			(xy 278.13 323.85) (xy 278.13 331.47)
-		)
-		(stroke
-			(width 0)
-			(type default)
-		)
-	)
-	(wire
-		(pts
 			(xy 234.95 297.18) (xy 234.95 298.45)
 		)
@@
 	(wire
 		(pts
-			(xy 316.23 322.58) (xy 316.23 331.47)
-		)
-		(stroke
-			(width 0)
-			(type default)
-		)
-	)
-	(wire
-		(pts
 			(xy 231.14 289.56) (xy 234.95 289.56)
 		)
@@
 	)
 	(symbol
-		(lib_id "power:+3V3")
-		(at 316.23 322.58 0)
-		(unit 1)
-		(exclude_from_sim no)
-		(in_bom yes)
-		(on_board yes)
-		(dnp no)
-		(fields_autoplaced yes)
-		(property "Reference" "#PWR097"
-			(at 316.23 326.39 0)
-			(effects
-				(font
-					(size 1.27 1.27)
-				)
-				(hide yes)
-			)
-		)
-		(property "Value" "+3V3"
-			(at 316.23 317.5 0)
-			(effects
-				(font
-					(size 1.27 1.27)
-				)
-			)
-		)
-		(property "Footprint" ""
-			(at 316.23 322.58 0)
-			(effects
-				(font
-					(size 1.27 1.27)
-				)
-				(hide yes)
-			)
-		)
-		(property "Datasheet" ""
-			(at 316.23 322.58 0)
-			(effects
-				(font
-					(size 1.27 1.27)
-				)
-				(hide yes)
-			)
-		)
-		(property "Description" ""
-			(at 316.23 322.58 0)
-			(effects
-				(font
-					(size 1.27 1.27)
-				)
-				(hide yes)
-			)
-		)
-		(pin "1"
-		)
-		(instances
-			(project "Carrier_Board"
-				(path "/3800e2ee-0692-4645-8143-10fd3578fa9c/acae2808-0785-47a5-82ee-45b1bca85a3e"
-					(reference "#PWR097")
-					(unit 1)
-				)
-			)
-		)
-	)
-	(symbol
 		(lib_id "Connector:TestPoint")
 		(at 129.54 215.9 90)
@@
 					(unit 1)
 				)
-			)
-		)
-	)
-	(symbol
-		(lib_id "power:+3V3")
-		(at 278.13 323.85 0)
-		(unit 1)
-		(exclude_from_sim no)
-		(in_bom yes)
-		(on_board yes)
-		(dnp no)
-		(fields_autoplaced yes)
-		(property "Reference" "#PWR088"
-			(at 278.13 327.66 0)
-			(effects
-				(font
-					(size 1.27 1.27)
-				)
-				(hide yes)
-			)
-		)
-		(property "Value" "+3V3"
-			(at 278.13 318.77 0)
-			(effects
-				(font
-					(size 1.27 1.27)
-				)
-			)
-		)
-		(property "Footprint" ""
-			(at 278.13 323.85 0)
-			(effects
-				(font
-					(size 1.27 1.27)
-				)
-				(hide yes)
-			)
-		)
-		(property "Datasheet" ""
-			(at 278.13 323.85 0)
-			(effects
-				(font
-					(size 1.27 1.27)
-				)
-				(hide yes)
-			)
-		)
-		(property "Description" ""
-			(at 278.13 323.85 0)
-			(effects
-				(font
-					(size 1.27 1.27)
-				)
-				(hide yes)
-			)
-		)
-		(pin "1"
-		)
-		(instances
-			(project "Carrier_Board"
-				(path "/3800e2ee-0692-4645-8143-10fd3578fa9c/acae2808-0785-47a5-82ee-45b1bca85a3e"
-					(reference "#PWR088")
-					(unit 1)
-				)
